File: pcb/binary-tree.kicad_pcb (KiCad board)
At the start: 2 copper layers, 50 x 50 mm, 30 parts, among them IC1 STM32F042K6T7, J1 MICROUSB, P2 SWD_TC, SW1 DFU, SW2 DPST, U1 MIC5504-3.3

Commit message: Routed reference board
Parts:
- moved J1 0.48 mm to (98.1, 107.3)
Connections:
- IC1 pad 10: (no net) -> /LED5
- IC1 pad 12: (no net) -> /LED6
- IC1 pad 13: (no net) -> /LED7
- IC1 pad 14: (no net) -> /LED8
- IC1 pad 6: (no net) -> /LED1
- IC1 pad 7: (no net) -> /LED2
- IC1 pad 8: (no net) -> /LED3
- IC1 pad 9: (no net) -> /LED4
- R2 pad 1: (no net) -> /LED1
- R3 pad 1: (no net) -> /LED2
- R4 pad 1: (no net) -> /LED3
- R5 pad 1: (no net) -> /LED4
- R6 pad 1: (no net) -> /LED5
- R7 pad 1: (no net) -> /LED6
- R8 pad 1: (no net) -> /LED7
- R9 pad 1: (no net) -> /LED8
Routing:
- net VCC: track 0.00 -> 86.4 mm
- net /LED4: track 0.00 -> 47.9 mm
- net GND: track 0.00 -> 43.7 mm, vias 0 -> 18
- net /LED1: track 0.00 -> 38.4 mm
- net /LED3: track 0.00 -> 36.7 mm, vias 0 -> 2
- net /LED8: track 0.00 -> 33.1 mm
- net /LED5: track 0.00 -> 28.2 mm
- net /LED7: track 0.00 -> 24.3 mm, vias 0 -> 2
- net /LED2: track 0.00 -> 21.4 mm
- net /USB_DM: track 0.00 -> 21.2 mm
- net /USB_DP: track 0.00 -> 21.1 mm
- net Net-(C4-Pad1): track 0.00 -> 20.7 mm
- net /LED6: track 0.00 -> 18.9 mm
- net Net-(IC1-Pad31): track 0.00 -> 16.6 mm
- net Net-(C7-Pad1): track 0.00 -> 13.6 mm
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- added copper zone on B.Cu, net GND
Other:
- net class Default: via_dia 0.6 -> 0.8
- rule via_min_size: 0.4 -> 0.8
- board text added: "2016-10-09"
- board text added: "DAVID TURNER"
- board text added: "GREEN"
- board text added: "MICROPROCESSOR"
- board text added: "ORANGE"
- board text added: "RED"
- board text added: "REFERENCE DESIGN"
- board text added: "USB CONNECTOR"
- board text added: "USB DFU"
- board text added: "USB PSU"
- board text added: "YELLOW"
